Commit message: 重大更新，使用xacro重新建模小车与机械臂，基本完成

File: urdf/car.xacro (robot description, xacro)
@@ -1,35 +1,175 @@
 <?xml version="1.0" encoding="utf-8"?>
-<robot name="car" xmlns:xacro="http://ros.org/wiki/xacro">
-    <xacro:property name="car_leng" value="0.386"/>
-    <xacro:property name="car_width" value="0.236"/>
+<robot name="arm_car" xmlns:xacro="http://ros.org/wiki/xacro">
+    <xacro:property name="car_leng" value="0.410"/>
+    <xacro:property name="car_width" value="0.238"/>
     <xacro:property name="car_height" value="0.06"/>
     <xacro:property name="car_mass" value="6.1"/>
-<link name="base_link">
-    <visual>
-      <origin rpy="0 0 0" xyz="0 0 0.05"/>
-      <geometry>
-        <box size="${car_leng} ${car_width} ${car_height}" />
-      </geometry>
-      <material name="">
-        <color rgba="0.8 0 1 1.0"/>
-      </material>
-    </visual>
-    <inertial>
-      <origin rpy="0 0 0" xyz="0 0 0.05"/>
-      <mass value="${car_mass}"/>
-      <inertia ixx="0.0425" ixy="0.0" ixz="0.0" iyy="0.1136" iyz="0.0" izz="0.1561" />
-    </inertial>
-    <collision>
-      <origin rpy="0 0 0" xyz="0 0 0.05" />
-      <geometry>
-        <box size="${car_leng} ${car_width} ${car_height}" />
-      </geometry>
-    </collision>
-</link>
-<link name="base"/>
-<joint name="base_base-link" type="fixed">
-  <origin rpy="0 0 0" xyz="0 0 0"/>
-  <parent link="base"/>
-  <child link="base_link"/>
-</joint>
+    <xacro:property name="PI" value="3.1415926535897931"/>
+    <xacro:property name="wheel_radius" value="0.05"/>
+    <xacro:property name="wheel_height" value="0.08"/>
+    <xacro:property name="wheel_mass" value="0.1"/>
+    <xacro:property name="camera_low_box_size" value="0.03"/>
+    <xacro:property name="laser_box_radius" value="0.03"/>
+    <xacro:property name="laser_box_height" value="0.03"/>
+    <xacro:property name="arm1_height" value="0.1"/>
+    <xacro:property name="arm1_radius" value="0.03"/>
+    <xacro:property name="arm1_mass" value="0.5"/>
+    <xacro:property name="arm2_height" value="0.2"/>
+    <xacro:property name="arm2_radius" value="0.02"/>
+    <xacro:property name="arm2_mass" value="0.3"/>
+    <xacro:property name="arm3_height" value="0.2"/>
+    <xacro:property name="arm3_radius" value="0.01"/>
+    <xacro:property name="arm3_mass" value="0.2"/>
+    <xacro:include filename="$(find npu_sim)/urdf/car.gazebo.xacro"/>
+    <xacro:macro name="wheel" params="wheel_name lr_reflect fb_reflect">
+        <link name="${wheel_name}_wheel">
+            <visual>
+                <origin rpy="0 0 0" xyz="0 0 0"/>
+                <geometry>
+                    <cylinder length="${wheel_height}" radius="${wheel_radius}"/>
+                </geometry>
+            </visual>
+            <inertial>
+                <mass value="${wheel_mass}" />
+                <inertia ixx="${wheel_mass*(3*wheel_radius*wheel_radius+wheel_height*wheel_height)/12.0}" ixy="0.0" ixz="0.0"
+                         iyy="${wheel_mass*(3*wheel_radius*wheel_radius+wheel_height*wheel_height)/12.0}" iyz="0.0"
+                         izz="${wheel_mass*wheel_radius*wheel_radius/2.0}" />
+            </inertial>
+            <collision>
+                <origin rpy="0 0 0" xyz="0 0 0" />
+                <geometry>
+                    <cylinder length="${wheel_height}" radius="${wheel_radius}"/>
+                </geometry>
+            </collision>
+        </link>
+        <joint name="base_${wheel_name}_joint" type="fixed">
+            <origin xyz="${0.156*fb_reflect} ${0.169*lr_reflect} -0.02" rpy="${PI/2} 0 0"/>
+            <parent link="base_link"/>
+            <child link="${wheel_name}_wheel"/>
+        </joint>
+    </xacro:macro>
+    <link name="footprint"/>
+    <joint name="foot_base_joint" type="fixed">
+        <origin xyz="0 0 0" rpy="0 0 0"/>
+        <parent link="footprint"/>
+        <child link="base_link"/>
+    </joint>
+    <link name="base_link">
+        <visual>
+          <origin rpy="0 0 0" xyz="0 0 0"/>
+          <geometry>
+            <box size="${car_leng} ${car_width} ${car_height}" />
+          </geometry>
+        </visual>
+        <inertial>
+          <mass value="${car_mass}"/>
+          <inertia ixx="0.0425" ixy="0.0" ixz="0.0" iyy="0.1136" iyz="0.0" izz="0.1561" />
+        </inertial>
+        <collision>
+          <origin rpy="0 0 0" xyz="0 0 0" />
+          <geometry>
+            <box size="${car_leng} ${car_width} ${car_height}" />
+          </geometry>
+        </collision>
+    </link>
+    <xacro:wheel wheel_name="left_front" lr_reflect="1" fb_reflect="1"/>
+    <xacro:wheel wheel_name="right_front" lr_reflect="-1" fb_reflect="1"/>
+    <xacro:wheel wheel_name="right_back" lr_reflect="-1" fb_reflect="-1"/>
+    <xacro:wheel wheel_name="left_back" lr_reflect="1" fb_reflect="-1"/>
+    <link name="imu_link"/>
+    <joint name="base_imu_joint" type="fixed">
+        <origin xyz="0 0 0" rpy="0 0 0"/>
+        <parent link="base_link"/>
+        <child link="imu_link"/>
+    </joint>
+    <joint name="base_laser_joint" type="fixed">
+        <origin xyz="0.1 0 ${(car_height+laser_box_height)/2}" rpy="0 0 0"/>
+        <parent link="base_link"/>
+        <child link="laser_link"/>
+    </joint>
+    <link name="laser_link">
+        <visual>
+            <origin rpy="0 0 0" xyz="0 0 0"/>
+            <geometry>
+                <cylinder radius="${laser_box_radius}" length="${laser_box_height}"/>
+            </geometry>
+        </visual>
+        <inertial>
+            <mass value="0.1"/>
+            <inertia ixx="${0.1*(3*laser_box_radius*laser_box_radius+laser_box_height*laser_box_height)/12.0}" ixy="0.0" ixz="0.0"
+                     iyy="${0.1*(3*laser_box_radius*laser_box_radius+laser_box_height*laser_box_height)/12.0}" iyz="0.0"
+                     izz="${0.1*laser_box_radius*laser_box_radius/2.0}" />
+        </inertial>
+    </link>
+    <joint name="base_camera_low_joint" type="continuous">
+        <axis xyz="0 1 0"/>
+        <origin xyz="${(car_leng-camera_low_box_size)/2} 0 ${(car_height+camera_low_box_size)/2}" rpy="0 0 0"/>
+        <parent link="base_link"/>
+        <child link="camera_low_link"/>
+    </joint>
+    <link name="camera_low_link">
+        <visual>
+            <origin rpy="0 0 0" xyz="0 0 0"/>
+            <geometry>
+                <box size="${camera_low_box_size} ${camera_low_box_size} ${camera_low_box_size}" />
+            </geometry>
+        </visual>
+        <inertial>
+            <mass value="0.05"/>
+            <inertia ixx="${0.05*camera_low_box_size*camera_low_box_size/6.0}" ixy="0.0" ixz="0.0"
+                     iyy="${0.05*camera_low_box_size*camera_low_box_size/6.0}" iyz="0.0"
+                     izz="${0.05*camera_low_box_size*camera_low_box_size/6.0}" />
+        </inertial>
+    </link>
+    <xacro:macro name="arm" params="joint_name last_arm_name arm_name z_shift radius height mass axis">
+        <joint name="${joint_name}" type="revolute">
+            <origin xyz="0 0 ${z_shift}" rpy="0 0 0"/>
+            <parent link="${last_arm_name}"/>
+            <child link="${arm_name}"/>
+            <axis xyz="${axis}"/>
+            <limit lower="-1" upper="1" effort="10.0" velocity="0.1"/>
+            <dynamics damping="0.3"/>
+<!--            damping big make some bug-->
+        </joint>
+        <link name="${arm_name}">
+            <visual>
+                <origin rpy="0 0 0" xyz="0 0 ${height/2}"/>
+                <geometry>
+                    <cylinder radius="${radius}" length="${height}"/>
+                </geometry>
+            </visual>
+            <inertial>
+                <origin rpy="0 0 0" xyz="0 0 ${height/2}"/>
+                <mass value="${mass}"/>
+                <inertia ixx="${mass*(3*radius*radius+height*height)/12.0}" ixy="0.0" ixz="0.0"
+                         iyy="${mass*(3*radius*radius+height*height)/12.0}" iyz="0.0"
+                         izz="${mass*radius*radius/2.0}" />
+            </inertial>
+        </link>
+    </xacro:macro>
+    <xacro:arm joint_name="base_arm1_joint" last_arm_name="base_link" arm_name="arm1_link" z_shift="${(car_height)/2}"
+               radius="${arm1_radius}" height="${arm1_height}" mass="${arm1_mass}" axis="0 0 1"/>
+    <xacro:arm joint_name="arm1_arm2_joint" last_arm_name="arm1_link" arm_name="arm2_link" z_shift="${arm1_height}"
+               radius="${arm2_radius}" height="${arm2_height}" mass="${arm2_mass}" axis="0 1 0"/>
+    <xacro:arm joint_name="arm2_arm3_joint" last_arm_name="arm2_link" arm_name="arm3_link" z_shift="${arm2_height}"
+               radius="${arm3_radius}" height="${arm3_height}" mass="${arm3_mass}" axis="0 1 0"/>
+    <joint name="arm3_camera_high_joint" type="fixed">
+        <origin xyz="${-camera_low_box_size/2-arm3_radius} 0 ${arm3_height/2}" rpy="0 ${-PI/2} 0"/>
+        <parent link="arm3_link"/>
+        <child link="camera_high_link"/>
+    </joint>
+    <link name="camera_high_link">
+        <visual>
+            <origin rpy="0 0 0" xyz="0 0 0"/>
+            <geometry>
+                <box size="${camera_low_box_size} ${camera_low_box_size} ${camera_low_box_size}" />
+            </geometry>
+        </visual>
+        <inertial>
+            <mass value="0.05"/>
+            <inertia ixx="${0.05*camera_low_box_size*camera_low_box_size/6.0}" ixy="0.0" ixz="0.0"
+                     iyy="${0.05*camera_low_box_size*camera_low_box_size/6.0}" iyz="0.0"
+                     izz="${0.05*camera_low_box_size*camera_low_box_size/6.0}" />
+        </inertial>
+    </link>
 </robot>
